File: Hardware/Kicad/battery_pwr_brd_r3.kicad_sch (KiCad schematic)
At the start: 31 parts, among them J1 INPUT_PWR, J2 Output_5V, J3 Output_3V3, Q2 MMBT3904, SW1 SW_DPDT_x2, U1 MCP1755, U2 LM1117MP-3.3

Commit message: Add files via upload
Parts:
- BT1: value CR2032 X 2 -> BATT HLD COIN 20MM 2 CELL PC PIN; Vendor (none) -> Digikey; Vendor Part# (none) -> BH800S-ND
- C1, C2, C7, C8: Vendor # 1276-1017-1-ND -> (none); Vendor Part# (none) -> 1276-1099-1-ND
- C3, C6: Vendor (none) -> Digikey; Vendor Part# (none) -> 1276-1244-1-ND
- C4, C5: Vendor (none) -> Digikey; Vendor Part# (none) -> 1276-1066-1-ND
- D1: value OC_Fault -> PWR_OK; Vendor Part # 1497-XZM2CRK55W-3RTCT-ND -> (none); Vendor Part# (none) -> 732-11422-1-ND
- D2, D4: value 1N5819WS -> 1N5819W; Vendor (none) -> Digikey; Vendor Part# (none) -> 1655-1N5819WCT-ND
- FB1: Vendor Part # 1934-1465-1-ND -> (none); Vendor Part# (none) -> 1934-1465-1-ND
- H1, H2, H3: now left out of the parts list
- J1: Vendor Part # CP-037A-ND -> (none); Vendor Part# (none) -> CP-037A-ND
- Q2: Vendor (none) -> Digikey; Vendor Part# (none) -> SMMBT3904LT3GOSCT-ND
- R1: Vendor (none) -> Digikey; Vendor Part# (none) -> 311-100KCRCT-ND
- R2: Vendor (none) -> Digiley; Vendor Part# (none) -> A126359CT-ND
- R3: Vendor (none) -> Digikey; Vendor Part# (none) -> 311-5.1KARCT-ND
- R4: Vendor (none) -> Digkey; Vendor Part# (none) -> 311-10.0KCRCT-ND
- SW1: Vendor (none) -> Digikey; Vendor Part# (none) -> 401-2002-1-ND
- SW1: footprint (none) -> jerrys_Library:SW_DPDT_CK_JS202011JCQN; Vendor (none) -> Digikey; Vendor Part# (none) -> 401-2002-1-ND
- U1: Vendor (none) -> Digikey; Vendor Part# (none) -> MCP1755ST-3302E/DBCT-ND
- U2: Vendor (none) -> Digikey; Vendor Part# (none) -> 497-1242-1-ND
